File: PCB's/aero_sense.kicad_sch (KiCad schematic)
At the start: 35 parts, among them J1 10164228-0201A1RLF, J2 10164228-0201A1RLF, J3 10164228-0201A1RLF, J4 10164228-0201A1RLF, U1 STM32F415ZGT6, U2 SHT45-AD1F-R2, U3 SGP41-D-R4, U4 MS560702BA03-00, U5 ICM-42688-P

Commit message: updatet liberys and added sensors to bottom pcb
Parts:
- added unit 2 of U1
- added unit 3 of U1
Connections:
- net VDDA: now also U1.33 (VDDA); no longer U1.33 (VDDA)
- net VDD_MCU: now also U1.108 (VDD), U1.121 (VDD), U1.131 (VDD), U1.144 (VDD), U1.17 (VDD), U1.30 (VDD), U1.39 (VDD), U1.52 (VDD), U1.62 (VDD), U1.72 (VDD), U1.84 (VDD), U1.95 (VDD); no longer U1.108 (VDD), U1.121 (VDD), U1.131 (VDD), U1.144 (VDD), U1.17 (VDD), U1.30 (VDD), U1.39 (VDD), U1.52 (VDD), U1.62 (VDD), U1.72 (VDD), U1.84 (VDD), U1.95 (VDD)
- net VREF+: now also U1.32 (VREF+); no longer U1.32 (VREF+)
- new net: U1.107 (VSS), U1.120 (VSS), U1.130 (VSS), U1.16 (VSS), U1.38 (VSS), U1.51 (VSS), U1.61 (VSS), U1.83 (VSS), U1.94 (VSS)
