File: PCB's/aero_sense.kicad_sch (KiCad schematic)
At the start: 0 parts

Commit message: Added connectors, started work on the schematic.
Parts:
- added C1, C12, C13, C14, C15, C16, C17, C18, C19, C2, C20, C21, C22, C23, C3, C4, C5, C6, C7, C8, C9: 100nF, Package_SO:SOIC-8_3.9x4.9mm_P1.27mm, symbol Device:C
- added C10, C11: 4.7uF, Package_SO:SOIC-8_3.9x4.9mm_P1.27mm, symbol Device:C
- added E1: ANT-GNSSCP-TH18L1, MyComponents:XCVR_ANT-GNSSCP-TH18L1, symbol Library:ANT-GNSSCP-TH18L1
- added FB1: FerriteBead, symbol Device:FerriteBead
- added J1, J2, J3, J4: 10164228-0201A1RLF, MyComponents:AMPHENOL_10164228-0201A1RLF, symbol Library:10164228-0201A1RLF
- added R1: R, Package_DIP:DIP-8_W7.62mm, symbol Device:R
- added U1: STM32F415ZGT6, MyComponents:LQFP144-20x20mm, symbol Library:STM32F415ZGT6
- added U2: SHT45-AD1F-R2, MyComponents:SHT4X, symbol Library:SHT45-AD1F-R2
- added U3: SGP41-D-R4, MyComponents:XDCR_SGP41-D-R4, symbol Library:SGP41-D-R4
- added U4: MS560702BA03-00, MyComponents:SON125P500X300X100-8N, symbol Library:MS560702BA03-00
- added U5: ICM-42688-P, MyComponents:PQFN50P300X250X97-14N, symbol Library:ICM-42688-P
Connections:
- net GND: now also C1.2, C10.2, C11.2, C12.2, C13.2, C14.2, C15.2, C16.2, C17.2, C18.2, C19.2, C2.2, C20.2, C21.2, C22.2, C23.2, C3.2, C4.2, C5.2, C6.2, C7.2, C8.2, C9.2
- new net: U4.4 (~{CSB}), U4.5 (~{CSB})
- new net: E1.2, E1.3, E1.4, E1.5
- new net: U1.107 (VSS), U1.120 (VSS), U1.130 (VSS), U1.16 (VSS), U1.38 (VSS), U1.51 (VSS), U1.61 (VSS), U1.83 (VSS), U1.94 (VSS)
- new net VDDA: FB1.1, R1.1, U1.33 (VDDA)
- new net VDD_MCU: C1.1, C10.1, C11.1, C12.1, C13.1, C14.1, C15.1, C16.1, C17.1, C18.1, C19.1, C2.1, C20.1, C21.1, C22.1, C23.1, C3.1, C4.1, C5.1, C6.1, C7.1, C8.1, C9.1, FB1.2, U1.108 (VDD), U1.121 (VDD), U1.131 (VDD), U1.144 (VDD), U1.17 (VDD), U1.30 (VDD), U1.39 (VDD), U1.52 (VDD), U1.62 (VDD), U1.72 (VDD), U1.84 (VDD), U1.95 (VDD)
- new net VREF+: R1.2, U1.32 (VREF+)

Commit message: added seperate sheets for power and bottom pcb
Other:
- added sheet Bottom PCB (bottom_pcb.kicad_sch)
- added sheet Power (power.kicad_sch)
Changed lines of the file:
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@@
+		)
+	)
+	(sheet
+		(at 317.5 177.8)
+		(size 355.6 203.2)
+		(exclude_from_sim no)
+		(in_bom yes)
+		(on_board yes)
+		(dnp no)
+		(fields_autoplaced yes)
+		(stroke
+			(width 0.1524)
+			(type solid)
+		)
+		(fill
+			(color 0 0 0 0)
+		)
+		(property "Sheetname" "Bottom PCB"
+			(at 317.5 177.0884 0)
+			(show_name no)
+			(do_not_autoplace no)
+			(effects
+				(font
+					(size 1.27 1.27)
+				)
+				(justify left bottom)
+			)
+		)
+		(property "Sheetfile" "bottom_pcb.kicad_sch"
+			(at 317.5 381.5846 0)
+			(show_name no)
+			(do_not_autoplace no)
+			(effects
+				(font
+					(size 1.27 1.27)
+				)
+				(justify left top)
+			)
+		)
+		(instances
+			(project "aero_sense"
+				(path "/4d06510f-84fa-43e7-942b-130a75a96407"
+					(page "2")
+				)
+			)
+		)
+	)
+	(sheet
+		(at 317.5 -11.43)
+		(size 354.33 182.88)
+		(exclude_from_sim no)
+		(in_bom yes)
+		(on_board yes)
+		(dnp no)
+		(fields_autoplaced yes)
+		(stroke
+			(width 0.1524)
+			(type solid)
+		)
+		(fill
+			(color 0 0 0 0)
+		)
+		(property "Sheetname" "Power"
+			(at 317.5 -12.1416 0)
+			(show_name no)
+			(do_not_autoplace no)
+			(effects
+				(font
+					(size 1.27 1.27)
+				)
+				(justify left bottom)
+			)
+		)
+		(property "Sheetfile" "power.kicad_sch"
+			(at 317.5 172.0346 0)
+			(show_name no)
+			(do_not_autoplace no)
+			(effects
+				(font
+					(size 1.27 1.27)
+				)
+				(justify left top)
+			)
+		)
+		(instances
+			(project "aero_sense"
+				(path "/4d06510f-84fa-43e7-942b-130a75a96407"
+					(page "3")
+				)
+			)
 		)
 	)

Commit message: updated power schematic
Parts:
- removed C1, C12, C13, C14, C15, C16, C17, C18, C19, C2, C20, C21, C22, C23, C3, C4, C5, C6, C7, C8, C9: 100nF, Package_SO:SOIC-8_3.9x4.9mm_P1.27mm, symbol Device:C
- removed C10, C11: 4.7uF, Package_SO:SOIC-8_3.9x4.9mm_P1.27mm, symbol Device:C
- removed E1: ANT-GNSSCP-TH18L1, MyComponents:XCVR_ANT-GNSSCP-TH18L1, symbol Library:ANT-GNSSCP-TH18L1
- removed FB1: FerriteBead, symbol Device:FerriteBead
- removed R1: R, Package_DIP:DIP-8_W7.62mm, symbol Device:R
- removed U2: SHT45-AD1F-R2, MyComponents:SHT4X, symbol Library:SHT45-AD1F-R2
- removed U3: SGP41-D-R4, MyComponents:XDCR_SGP41-D-R4, symbol Library:SGP41-D-R4
- removed U4: MS560702BA03-00, MyComponents:SON125P500X300X100-8N, symbol Library:MS560702BA03-00
Connections:
- removed net VDDA: U1.33 (VDDA)
- removed net VDD_MCU: U1.108 (VDD), U1.121 (VDD), U1.131 (VDD), U1.144 (VDD), U1.17 (VDD), U1.30 (VDD), U1.39 (VDD), U1.52 (VDD), U1.62 (VDD), U1.72 (VDD), U1.84 (VDD), U1.95 (VDD)
- removed net VREF+: U1.32 (VREF+)
Other:
- moved on the sheet: U5
