File: PCB's/bottom_pcb.kicad_sch (KiCad schematic)
At the start: 3 parts, among them U6 BMP581, U7 SHT45-AD1F-R2, U8 SGP41-D-R4

Commit message: Revert "Merge branch 'main' of https://github.com/AlexElman/Aero_sense"
This reverts commit 38703e91a3bcee96153a0bc5ec74bb509ab77a91, reversing
changes made to ef282aac22077f3b7d244ed21cf80990a026c3e9.
Parts:
- removed U6: BMP581, QFN10_BMP581_BOS, symbol Library:BMP581
- removed U7: SHT45-AD1F-R2, SHT45-AD1F-R2:SHT4X, symbol Library:SHT45-AD1F-R2
- removed U8: SGP41-D-R4, SGP41-D-R4:XDCR_SGP41-D-R4, symbol Library:SGP41-D-R4

Commit message: updatet liberys and added sensors to bottom pcb
Parts:
- added U6: BMP581, QFN10_BMP581_BOS, symbol Library:BMP581
- added U7: SHT45-AD1F-R2, SHT45-AD1F-R2:SHT4X, symbol Library:SHT45-AD1F-R2
- added U8: SGP41-D-R4, SGP41-D-R4:XDCR_SGP41-D-R4, symbol Library:SGP41-D-R4
