File: PCB's/power.kicad_sch (KiCad schematic)
At the start: 32 parts, among them U1 STM32F415ZGT6

Commit message: pcb
Parts:
- removed C1, C12, C13, C14, C15, C16, C17, C18, C19, C2, C20, C21, C22, C23, C24, C28, C3, C4, C5, C6, C7, C8, C9: 100nF, Capacitor_SMD:C_0201_0603Metric, symbol Device:C
- removed C10, C11: 4.7uF, Capacitor_SMD:C_0201_0603Metric, symbol Device:C
- removed C25, C26: 2uF, Capacitor_SMD:C_0201_0603Metric, symbol Device:C
- removed C27, C29: 1uF, Capacitor_SMD:C_0201_0603Metric, symbol Device:C
- removed FB1: FerriteBead, symbol Device:FerriteBead
- removed R1: 0R, Resistor_SMD:R_0201_0603Metric, symbol Device:R
- removed U1: STM32F415ZGT6, MyComponents:LQFP144-20x20mm, symbol Library:STM32F415ZGT6
Other:
- note removed: "Ceramic Capacitors low ESR"

Commit message: fixed power schematic merge conflict
Parts:
- added C1, C12, C13, C14, C15, C16, C17, C18, C19, C2, C20, C21, C22, C23, C24, C28, C3, C4, C5, C6, C7, C8, C9: 100nF, Capacitor_SMD:C_0201_0603Metric, symbol Device:C
- added C10, C11: 4.7uF, Capacitor_SMD:C_0201_0603Metric, symbol Device:C
- added C25, C26: 2uF, Capacitor_SMD:C_0201_0603Metric, symbol Device:C
- added C27, C29: 1uF, Capacitor_SMD:C_0201_0603Metric, symbol Device:C
- added FB1: FerriteBead, symbol Device:FerriteBead
- added R1: 0R, Resistor_SMD:R_0201_0603Metric, symbol Device:R
- added U1: STM32F415ZGT6, MyComponents:LQFP144-20x20mm, symbol Library:STM32F415ZGT6
Connections:
- new net: C26.1, U1.71 (VCAP_1)
- new net: C25.1, U1.106 (VCAP_2)
- new net GND: C1.2, C10.2, C11.2, C12.2, C13.2, C14.2, C15.2, C16.2, C17.2, C18.2, C19.2, C2.2, C20.2, C21.2, C22.2, C23.2, C24.2, C25.2, C26.2, C27.2, C28.2, C29.2, C3.2, C4.2, C5.2, C6.2, C7.2, C8.2, C9.2, U1.107 (VSS), U1.120 (VSS), U1.130 (VSS), U1.16 (VSS), U1.31 (VSSA), U1.38 (VSS), U1.51 (VSS), U1.61 (VSS), U1.83 (VSS), U1.94 (VSS)
- new net VDDA: C27.1, C28.1, FB1.1, R1.1, U1.33 (VDDA)
- new net VDD_MCU: C1.1, C10.1, C11.1, C12.1, C13.1, C14.1, C15.1, C16.1, C17.1, C18.1, C19.1, C2.1, C20.1, C21.1, C22.1, C23.1, C3.1, C4.1, C5.1, C6.1, C7.1, C8.1, C9.1, FB1.2, U1.108 (VDD), U1.121 (VDD), U1.131 (VDD), U1.144 (VDD), U1.17 (VDD), U1.30 (VDD), U1.39 (VDD), U1.52 (VDD), U1.62 (VDD), U1.72 (VDD), U1.84 (VDD), U1.95 (VDD)
- new net VREF+: C24.1, C29.1, R1.2, U1.32 (VREF+)
Other:
- note added: "Ceramic Capacitors low ESR"
