File: PCB's/power.kicad_sch (KiCad schematic)
At the start: 32 parts, among them U1 STM32F415ZGT6

Commit message: added top pcb hierarchical sheet and updated power schematic
Parts:
- added C24: 100nF, Capacitor_SMD:C_0201_0603Metric, symbol Device:C
- U9: renamed from U1; footprint MyComponents:LQFP144-20x20mm -> (none)
- renumbered C1 to C28, C12 to C29, C28 to C30, C2 to C31, C13 to C32, C24 to C33, C3 to C34, C14 to C35, C29 to C36, C4 to C37, C15 to C38, C5 to C39, C16 to C40, C6 to C41, C17 to C42, C7 to C43, C18 to C44, C8 to C45, C19 to C46, C9 to C47, C20 to C48, C21 to C49, C10 to C50, C22 to C51, C11 to C52, C23 to C53, FB1 to FB2, R1 to R2
Connections:
- net GND: now also C24.2
- net VDD_MCU: now also U9.6 (VBAT), C24.1
Other:
- note added: "test123"
- moved on the sheet: C25, C26, U9C
