File: PCB's/top_pcb.kicad_sch (KiCad schematic)
At the start: 0 parts

Commit message: cleaner liberary and unfinished top pcb
Parts:
- added J7: 10164227-0205A1RLF, 10164227-0205A1RLF:AMPHENOL_10164227-0205A1RLF, symbol Library:10164227-0205A1RLF
- added J8: Conn_01x04_Pin, Connector:Tag-Connect_TC2030-IDC-FP_2x03_P1.27mm_Vertical, symbol Connector:Conn_01x04_Pin
- added U10: SAM-M10Q-00B, SAM-M10Q_UBL, symbol Library:SAM-M10Q-00B
Connections:
- new net +3.3V: U10.17 (VCC), U10.2 (V_IO)
- new net +5V: J8.2 (Pin_2)
- new net GND: J8.1 (Pin_1), U10.1 (GND), U10.10 (GND), U10.11 (GND), U10.15 (GND), U10.16 (GND), U10.20 (GND), U10.4 (GND), U10.5 (GND), U10.6 (GND)
Other:
- note added: "Anschluesse fuer MicoAir LR868F"
- note added: "SDA offen = I²C nicht genutzt"
